Commit message: Change Lidar Size

File: urdf/unified_radars.urdf (robot description, URDF)
Before this commit: robot morning_car, 3 links, 2 joints
Links:
- link RADARS: geometry visual box size=0.01 0.01 0.01
- link hesai_lidar: geometry visual cylinder length=0.04845 radius=0.059
Joints:
- joint base_roof_lidar: origin xyz=0.716 -0.189 0 rpy=0 0 0 -> xyz=0 0 0.2777 rpy=0 0 0
